File: E-ink Display Progammer.kicad_pcb (KiCad board)
At the start: 2 copper layers, 85.7 x 71.7 mm, 56 parts, among them IC1 TXS0108E, J1 Conn_01x08_Male, J2 Conn_01x06_Female, J3 Conn_01x06_Female

Commit message: rev 1.1
Parts:
- J2, J3: footprint Connector_PinHeader_2.54mm:PinHeader_1x06_P2.54mm_Vertical -> AeonLabs:pogo 6pin magnetic
- moved G*** 61.9 mm to (175.7, 141.9)
- moved G*** 33.2 mm to (110.3, 134.6)
- moved IDSDA1 28.7 mm to (151.1, 131.0), turned to -90 degrees
- moved IDSCK1 26.8 mm to (148.6, 131.0), turned to -90 degrees
- moved IDMOSI1 25.2 mm to (146.0, 131.0), turned to -90 degrees
- moved ID3V3 24.9 mm to (133.2, 131.0), turned to -90 degrees
- moved IDMISO1 24.1 mm to (143.4, 131.0), turned to -90 degrees
- moved IDRST1 23.9 mm to (135.8, 131.0), turned to -90 degrees
- moved IDGND1 23.4 mm to (138.4, 131.0), turned to -90 degrees
- moved G*** 22.6 mm to (179.9, 161.3)
- moved BUZZER1 8.32 mm to (121.1, 89.3)
- moved FPC1 7.55 mm to (145.1, 86.5)
- moved FPC2 7.55 mm to (152.6, 87.8)
- moved FPC3 7.55 mm to (143.1, 92.9)
- moved FPD1 7.55 mm to (138.2, 86.8)
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Routing:
- net /GND: track 243.4 -> 286.0 mm, vias 12 -> 14
- net /IO23_RF_MOSI: track 63.1 -> 29.4 mm
- net /IO04_RF_SDA: track 69.5 -> 41.8 mm
- net /IO18_RF_SCK: track 65.3 -> 39.5 mm
- net /IO22_RF_RST: track 88.0 -> 73.0 mm
- net /IO21_RF_MISO: track 88.5 -> 73.5 mm, vias 2 -> 3
- net /IO12_LED_G: track 77.9 -> 89.8 mm
- net /IO14_LED_B: track 82.4 -> 92.2 mm
- net /IO13_LED_R: track 75.2 -> 84.5 mm
- net /IO19_EINK_BUSY: track 16.3 -> 23.8 mm
- net /IO17_EINK_RES: track 11.4 -> 19.0 mm
- net /IO16_EINK_CS: track 8.88 -> 16.0 mm
- net /RESE: track 28.6 -> 35.6 mm
- net /IO0_BOOT_DTR: track 93.4 -> 97.9 mm
- net /TX_IN: track 78.1 -> 82.3 mm
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Other:
- outline, holes or cut-outs redrawn
- board text added: "38 mm"
- board text added: "73x86mm board rev. 1.1 made to Fit a 2.5{dblquote} HDD case"
- board text added: "WIFI BLE RFID NFC contactless E-Ink Display Programmer Magnetic Pogo Pins"
- board text removed: "46.8mm"
- board text removed: "73x86mm board rev. 1.0 made to Fit a 2.5{dblquote} HDD case"
- board text removed: "WIFI BLE RFID NFC contactless E-Ink Display Programmer magnetic pogo pins"
