File: E-ink Display Progammer.kicad_sch (KiCad schematic)
At the start: 49 parts, among them IC1 TXS0108E, J1 Conn_01x08_Male, J2 Conn_01x06_Female, J3 Conn_01x06_Female

Commit message: rev 1.1
Parts:
- J2, J3: footprint Connector_PinHeader_2.54mm:PinHeader_1x06_P2.54mm_Vertical -> AeonLabs:pogo 6pin magnetic
Changed lines of the file:
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@@
       (effects (font (size 1.27 1.27)) (justify left))
     )
-    (property "Footprint" "Connector_PinHeader_2.54mm:PinHeader_1x06_P2.54mm_Vertical" (id 2) (at 275.336 120.904 0)
+    (property "Footprint" "AeonLabs:pogo 6pin magnetic" (id 2) (at 275.336 120.904 0)
       (effects (font (size 1.27 1.27)) hide)
     )
@@
       (effects (font (size 1.27 1.27)) (justify left))
     )
-    (property "Footprint" "Connector_PinHeader_2.54mm:PinHeader_1x06_P2.54mm_Vertical" (id 2) (at 275.59 154.686 0)
+    (property "Footprint" "AeonLabs:pogo 6pin magnetic" (id 2) (at 275.59 154.686 0)
       (effects (font (size 1.27 1.27)) hide)
     )
@@
     )
     (path "/6e89e1a9-de4b-4233-bf27-a064488a3d9d"
-      (reference "J2") (unit 1) (value "Conn_01x06_Female") (footprint "Connector_PinHeader_2.54mm:PinHeader_1x06_P2.54mm_Vertical")
+      (reference "J2") (unit 1) (value "Conn_01x06_Female") (footprint "AeonLabs:pogo 6pin magnetic")
     )
     (path "/9d330f3f-3613-4fb7-ac40-e8afc5072b0c"
-      (reference "J3") (unit 1) (value "Conn_01x06_Female") (footprint "Connector_PinHeader_2.54mm:PinHeader_1x06_P2.54mm_Vertical")
+      (reference "J3") (unit 1) (value "Conn_01x06_Female") (footprint "AeonLabs:pogo 6pin magnetic")
     )
     (path "/00000000-0000-0000-0000-00006187cf6b"
